File: PCBs/Controller/Controller.kicad_sch (KiCad schematic)
At the start: 62 parts, among them J1 USB_B_Micro, J2 Micro_SD_Card_Det1, J3 RS485, J4 UART, J5 TagConnect, Q1 PMOS, SW1 NSRT Swtich, SW2 NSRT Swtich, U1 STM32F030R8Tx, U2 TPS62125DSG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

Commit message: kicad changes
Parts:
- removed C3, C7: 10u, Capacitor_SMD:C_0603_1608Metric, symbol Device:C
- removed J1: USB_B_Micro, 4022S:microUSB, symbol Connector:USB_B_Micro
- removed JP1: ReversePolarity, Jumper:SolderJumper-2_P1.3mm_Open_TrianglePad1.0x1.5mm, symbol Jumper:SolderJumper_2_Open
- removed JP2: SolderJumper_2_Open, Jumper:SolderJumper-2_P1.3mm_Open_TrianglePad1.0x1.5mm, symbol Jumper:SolderJumper_2_Open
- removed L1, L2, L3: 4.7u, Inductor_SMD:L_0603_1608Metric, symbol Device:L
- removed Q1: PMOS, Package_TO_SOT_SMD:SOT-23, symbol Transistor_FET:AO3401A
- removed R2: 100k, Resistor_SMD:R_0603_1608Metric, symbol Device:R
- removed R6: 4.7M, Resistor_SMD:R_0603_1608Metric, symbol Device:R
- removed R7: 1.5M, Resistor_SMD:R_0603_1608Metric, symbol Device:R
- removed TP1: 5V, TestPoint:TestPoint_THTPad_2.0x2.0mm_Drill1.0mm, symbol Connector:TestPoint
- removed U2: TPS62125DSG, Package_SON:WSON-8-1EP_2x2mm_P0.5mm_EP0.9x1.6mm, symbol Regulator_Switching:TPS62125DSG
- SW1, SW2: value NSRT Swtich -> Switch
Connections:
- no-connect marks 16 -> 13
Other:
- note removed: "3.3V"
- note removed: "5V"
