File: PCBs/GoldElectrode/GoldElectrode.kicad_pcb (KiCad board)
At the start: 2 copper layers, 30 x 50.5 mm, 2 parts, among them J1 Finger, J2 Pad

Commit message: pcb work
Other:
- board size 30 x 50.5 mm -> 30 x 51 mm
Changed lines of the file:
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@@
-	)
-	(gr_arc
-		(start 97.5 57.5)
-		(mid 96.767767 59.267767)
-		(end 95 60)
-		(stroke
-			(width 0.05)
-			(type default)
-		)
-		(layer "Edge.Cuts")
 	)
 	(gr_arc
@@
 	)
 	(gr_line
-		(start 97.5 42)
-		(end 97.5 57.5)
-		(stroke
-			(width 0.05)
-			(type default)
-		)
-		(layer "Edge.Cuts")
-	)
-	(gr_line
-		(start 100 39.5)
-		(end 110 39.5)
+		(start 101.5 40)
+		(end 101.5 57.5)
+		(stroke
+			(width 0.05)
+			(type default)
+		)
+		(layer "Edge.Cuts")
+	)
+	(gr_line
+		(start 102.5 39)
+		(end 107.5 39)
 		(stroke
 			(width 0.05)
@@
 		(layer "Edge.Cuts")
 	)
+	(gr_arc
+		(start 111 60)
+		(mid 109.232233 59.267767)
+		(end 108.5 57.5)
+		(stroke
+			(width 0.05)
+			(type default)
+		)
+		(layer "Edge.Cuts")
+	)
+	(gr_line
+		(start 111 60)
+		(end 115 60)
+		(stroke
+			(width 0.05)
+			(type default)
+		)
+		(layer "Edge.Cuts")
+	)
 	(gr_line
 		(start 95 90)
@@
 	)
 	(gr_line
-		(start 112.5 42)
-		(end 112.5 57.5)
-		(stroke
-			(width 0.05)
-			(type default)
-		)
-		(layer "Edge.Cuts")
-	)
-	(gr_arc
-		(start 110 39.5)
-		(mid 111.767767 40.232233)
-		(end 112.5 42)
+		(start 108.5 40)
+		(end 108.5 57.5)
+		(stroke
+			(width 0.05)
+			(type default)
+		)
+		(layer "Edge.Cuts")
+	)
+	(gr_arc
+		(start 101.5 57.5)
+		(mid 100.767767 59.267767)
+		(end 99 60)
+		(stroke
+			(width 0.05)
+			(type default)
+		)
+		(layer "Edge.Cuts")
+	)
+	(gr_line
+		(start 95 60)
+		(end 99 60)
 		(stroke
 			(width 0.05)
@@
 	)
 	(gr_arc
-		(start 97.5 42)
-		(mid 98.232233 40.232233)
-		(end 100 39.5)
-		(stroke
-			(width 0.05)
-			(type default)
-		)
-		(layer "Edge.Cuts")
-	)
-	(gr_arc
-		(start 115 60)
-		(mid 113.232233 59.267767)
-		(end 112.5 57.5)
+		(start 107.5 39)
+		(mid 108.207107 39.292893)
+		(end 108.5 40)
 		(stroke
 			(width 0.05)
@@
 		(layer "Edge.Cuts")
 	)
+	(gr_arc
+		(start 101.5 40)
+		(mid 101.792893 39.292893)
+		(end 102.5 39)
+		(stroke
+			(width 0.05)
+			(type default)
+		)
+		(layer "Edge.Cuts")
+	)
+	(dimension
+		(type aligned)
+		(layer "Edge.Cuts")
+		(pts
+			(xy 101.5 44.5) (xy 108.5 44.5)
+		)
+		(height -9.25)
+		(gr_text "7.0000 mm"
+			(at 105 34.1 0)
+			(layer "Edge.Cuts")
+			(effects
+				(font
+					(size 1 1)
+					(thickness 0.15)
+				)
+			)
+		)
+		(format
+			(prefix "")
+			(suffix "")
+			(units 3)
+			(units_format 1)
+			(precision 4)
+		)
+		(style
+			(thickness 0.05)
+			(arrow_length 1.27)
+			(text_position_mode 0)
+			(extension_height 0.58642)
+			(extension_offset 0.5) keep_text_aligned)
+	)
+	(dimension
+		(type aligned)
+		(layer "Edge.Cuts")
+		(pts
+			(xy 102.5 43.25) (xy 107.5 43.25)
+		)
+		(height -5.5)
+		(gr_text "5.0000 mm"
+			(at 105 36.6 0)
+			(layer "Edge.Cuts")
+			(effects
+				(font
+					(size 1 1)
+					(thickness 0.15)
+				)
+			)
+		)
+		(format
+			(prefix "")
+			(suffix "")
+			(units 3)
+			(units_format 1)
+			(precision 4)
+		)
+		(style
+			(thickness 0.05)
+			(arrow_length 1.27)
+			(text_position_mode 0)
+			(extension_height 0.58642)
+			(extension_offset 0.5) keep_text_aligned)
+	)
 	(segment

Commit message: kicad changes
Parts:
- removed J1: Finger, 4022S:Finger_01
- removed J2: Pad, 4022S:Pad_20x20_mm
- added J3: Pad, 4022S:Gold_electrode_pad, F.Cu at (109.0, 76.0)
- added J4: Finger, 4022S:Gold_electrode_finger, F.Cu at (109.0, 53.5)
Routing:
- net Net-(J1-Pin_1): track 25.1 -> 0.00 mm
- net /Pad: track 0.00 -> 23.0 mm
- net /Fringe Shield: track 0.00 -> 22.0 mm
Other:
- board size 30 x 51 mm -> 28 x 40 mm
