File: PCBs/Probe/Probe.kicad_pcb (KiCad board)
At the start: 4 copper layers, 0 parts

Commit message: pcb work
Parts:
- added C1: 2.2u, Capacitor_SMD:C_0603_1608Metric, F.Cu at (124.8, 81.0)
- added C10: 100n, Capacitor_SMD:C_0603_1608Metric, F.Cu at (130.8, 66.0)
- added C11: 100n, Capacitor_SMD:C_0603_1608Metric, F.Cu at (132.2, 66.0)
- added C12: 100n, Capacitor_SMD:C_0603_1608Metric, F.Cu at (119.2, 61.5)
- added C13: 100n, Capacitor_SMD:C_0603_1608Metric, F.Cu at (119.2, 63.0)
- added C14: 100n, Capacitor_SMD:C_0603_1608Metric, F.Cu at (124.8, 92.1)
- added C15: 100n, Capacitor_SMD:C_0603_1608Metric, F.Cu at (147.5, 76.2)
- added C16: 100n, Capacitor_SMD:C_0603_1608Metric, F.Cu at (147.5, 77.8)
- added C2: 100n, Capacitor_SMD:C_0603_1608Metric, F.Cu at (115.8, 72.5)
- added C3: 2.2u, Capacitor_SMD:C_0603_1608Metric, F.Cu at (124.8, 79.5)
- added C4: 10u, Capacitor_SMD:C_0603_1608Metric, F.Cu at (104.0, 64.2)
- added C5: 1u, Capacitor_SMD:C_0603_1608Metric, F.Cu at (114.2, 72.5)
- added C6: 4.7u, Capacitor_SMD:C_0603_1608Metric, F.Cu at (124.8, 78.0)
- added C7: 100n, Capacitor_SMD:C_0603_1608Metric, F.Cu at (127.8, 78.0)
- added C8: 100n, Capacitor_SMD:C_0603_1608Metric, F.Cu at (127.8, 79.5)
- added C9: 4.7u, Capacitor_SMD:C_0603_1608Metric, F.Cu at (119.8, 78.0)
- added D1: GREEN, LED_SMD:LED_0805_2012Metric, F.Cu at (120.0, 80.8)
- added D2: RED, LED_SMD:LED_0603_1608Metric, F.Cu at (118.0, 81.0)
- added J1: Au+1, 4022S:Au_Electrode, B.Cu at (118.8, 94.2)
- added J10: TagConnect, Connector:Tag-Connect_TC2030-IDC-NL_2x03_P1.27mm_Vertical, B.Cu at (139.2, 58.8)
- added J2: Au+2, 4022S:Au_Electrode, B.Cu at (115.6, 94.2)
- added J3: Ti+, Connector_PinHeader_2.54mm:PinHeader_1x01_P2.54mm_Vertical, B.Cu at (140.1, 94.1)
- added J4: Au-1, 4022S:Au_Electrode, B.Cu at (131.5, 94.2)
- added J5: Au-2, 4022S:Au_Electrode, B.Cu at (103.1, 94.2)
- added J6: Ti-1, Connector_PinHeader_2.54mm:PinHeader_1x01_P2.54mm_Vertical, B.Cu at (135.1, 94.1)
- added J7: Ti-2, Connector_PinHeader_2.54mm:PinHeader_1x01_P2.54mm_Vertical, B.Cu at (145.2, 94.1)
- added J8: Debug, Connector_PinSocket_2.54mm:PinSocket_1x04_P2.54mm_Vertical, B.Cu at (140.5, 52.8)
- added J9: RS485, Connector_PinSocket_2.54mm:PinSocket_1x04_P2.54mm_Vertical, B.Cu at (128.6, 52.7)
- added JP1: FB, Jumper:SolderJumper-3_P2.0mm_Open_TrianglePad1.0x1.5mm, B.Cu at (106.2, 63.8)
- added JP2: ReversePolarity, Jumper:SolderJumper-2_P1.3mm_Open_TrianglePad1.0x1.5mm, B.Cu at (132.1, 57.5)
- added JP3: ReversePolarity, Jumper:SolderJumper-2_P1.3mm_Open_TrianglePad1.0x1.5mm, B.Cu at (127.3, 57.5)
- added Q1: S8050_SMD, Package_TO_SOT_SMD:SOT-23-3, F.Cu at (109.2, 62.5)
- added Q2: PMOS, Package_TO_SOT_SMD:SOT-23, F.Cu at (132.1, 57.5)
- added Q3: PMOS, Package_TO_SOT_SMD:SOT-23, F.Cu at (127.3, 57.5)
- added R1: 10k, Resistor_SMD:R_0603_1608Metric, F.Cu at (121.5, 62.2)
- added R10: 3k, Resistor_SMD:R_0603_1608Metric, F.Cu at (105.2, 78.8)
- added R11: 30k, Resistor_SMD:R_0603_1608Metric, F.Cu at (105.2, 83.2)
- added R12: 300, Resistor_SMD:R_0603_1608Metric, F.Cu at (105.2, 75.8)
- added R13: 3k, Resistor_SMD:R_0603_1608Metric, F.Cu at (105.2, 80.2)
- added R14: 30k, Resistor_SMD:R_0603_1608Metric, F.Cu at (105.2, 84.8)
- added R15: 120, Resistor_SMD:R_0603_1608Metric, F.Cu at (117.2, 56.0)
- added R16: 300, Resistor_SMD:R_0603_1608Metric, F.Cu at (105.2, 77.2)
- added R17: 3k, Resistor_SMD:R_0603_1608Metric, F.Cu at (105.2, 81.8)
- added R18: 30k, Resistor_SMD:R_0603_1608Metric, F.Cu at (105.2, 86.2)
- added R19: 1k, Resistor_SMD:R_1206_3216Metric, F.Cu at (143.8, 83.2)
- added R2: 4.7k, Resistor_SMD:R_0603_1608Metric, F.Cu at (114.2, 65.5)
- added R20: 10k, Resistor_SMD:R_1206_3216Metric, F.Cu at (146.8, 83.2)
- added R21: 1k, Resistor_SMD:R_0603_1608Metric, F.Cu at (120.0, 84.0)
- added R22: 1k, Resistor_SMD:R_0603_1608Metric, F.Cu at (118.0, 84.0)
- added R3: 4.7k, Resistor_SMD:R_0603_1608Metric, F.Cu at (115.8, 65.5)
- added R4: 20, Resistor_SMD:R_0603_1608Metric, F.Cu at (110.8, 85.8)
- added R5: 20, Resistor_SMD:R_0603_1608Metric, F.Cu at (110.8, 84.2)
- added R6: 20, Resistor_SMD:R_0603_1608Metric, F.Cu at (110.8, 82.8)
- added R7: 20, Resistor_SMD:R_0603_1608Metric, F.Cu at (110.8, 81.2)
- added R8: 10k, Resistor_SMD:R_0603_1608Metric, F.Cu at (112.8, 52.5)
- added R9: 300, Resistor_SMD:R_0603_1608Metric, F.Cu at (105.2, 74.2)
- added TP10: UBDAC, TestPoint:TestPoint_THTPad_2.0x2.0mm_Drill1.0mm, B.Cu at (135.8, 69.0)
- added TP11: DAC, TestPoint:TestPoint_THTPad_2.0x2.0mm_Drill1.0mm, B.Cu at (138.8, 69.0)
- added TP12: AMP, TestPoint:TestPoint_THTPad_2.0x2.0mm_Drill1.0mm, B.Cu at (141.8, 69.0)
- added TP13: SIG, TestPoint:TestPoint_THTPad_2.0x2.0mm_Drill1.0mm, B.Cu at (144.8, 69.0)
- added TP14: CALIB, TestPoint:TestPoint_THTPad_2.0x2.0mm_Drill1.0mm, B.Cu at (147.8, 69.0)
- added TP15: GND, TestPoint:TestPoint_THTPad_2.0x2.0mm_Drill1.0mm, B.Cu at (147.8, 59.2)
- added TP5: SCL, TestPoint:TestPoint_THTPad_2.0x2.0mm_Drill1.0mm, B.Cu at (135.8, 64.1)
- added TP6: SDA, TestPoint:TestPoint_THTPad_2.0x2.0mm_Drill1.0mm, B.Cu at (138.8, 64.1)
- added TP7: RS485_UART, TestPoint:TestPoint_THTPad_2.0x2.0mm_Drill1.0mm, B.Cu at (141.8, 64.1)
- added TP8: RS485_DE, TestPoint:TestPoint_THTPad_2.0x2.0mm_Drill1.0mm, B.Cu at (144.8, 64.1)
- added TP9: 3V3, TestPoint:TestPoint_THTPad_2.0x2.0mm_Drill1.0mm, B.Cu at (147.8, 64.1)
- added U1: ~, Package_SON:WSON-8-1EP_2x2mm_P0.5mm_EP0.9x1.6mm, F.Cu at (104.1, 62.2)
- added U2: STM32F401RCTx, Package_QFP:LQFP-64_10x10mm_P0.5mm, F.Cu at (123.2, 70.5)
- added U3: ~, Package_SO:TSSOP-14_4.4x5mm_P0.65mm, F.Cu at (107.0, 68.8)
- added U4: SP3485EN, Package_SO:SOIC-8_3.9x4.9mm_P1.27mm, F.Cu at (112.8, 56.0)
- added U5: OP07C, Package_SO:SOIC-8_3.9x4.9mm_P1.27mm, F.Cu at (144.8, 88.4)
- added U6: ~, Package_SO:TSSOP-14_4.4x5mm_P0.65mm, F.Cu at (111.0, 77.2)
- added U7: ~, Package_CSP:WLCSP-8_1.551x2.284mm_P0.5mm, F.Cu at (124.8, 94.8)
- added U8: ~, Package_SO:TSSOP-14_4.4x5mm_P0.65mm, F.Cu at (135.6, 83.7)
- added U9: ~, 4022S:WF183DE, F.Cu at (140.2, 76.0)
Routing:
- net /AMP: track 0.00 -> 100.1 mm, vias 0 -> 2
- net /SDA: track 0.00 -> 98.4 mm, vias 0 -> 6
- net /SCL: track 0.00 -> 98.3 mm, vias 0 -> 7
- net GND: track 0.00 -> 85.2 mm, vias 0 -> 19
- net /Calibration: track 0.00 -> 71.1 mm, vias 0 -> 4
- net /Ti-: track 0.00 -> 68.3 mm, vias 0 -> 3
- net /Au-: track 0.00 -> 68.2 mm, vias 0 -> 4
- net /Au+: track 0.00 -> 66.9 mm, vias 0 -> 3
- net /SIGNAL: track 0.00 -> 66.0 mm, vias 0 -> 2
- net /Ti+: track 0.00 -> 61.0 mm, vias 0 -> 3
- net +3V3: track 0.00 -> 58.7 mm, vias 0 -> 16
- net /DAC: track 0.00 -> 55.2 mm, vias 0 -> 5
- net /UNBUFF_DAC: track 0.00 -> 50.5 mm, vias 0 -> 3
- net /RS485_uart: track 0.00 -> 50.0 mm, vias 0 -> 3
- net /RS485_DE: track 0.00 -> 48.9 mm, vias 0 -> 3
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- added copper zone on In1.Cu, net +3V3
- added copper zone on In2.Cu, net GND
Other:
- board outline added: 50 x 50 mm
- board text added: "+"
- board text added: "3V3"
- board text added: "3v3"
- board text added: "A"
- board text added: "B"
- board text added: "BUFF"
- board text added: "Debug RP"
- board text added: "FB"
- board text added: "GND"
- board text added: "RS485"
- board text added: "RS485 RP"
- board text added: "Rx"
- board text added: "Tx"
- board text added: "UART"
- board text added: "UNBUFF"
- board text added: "amp"
- board text added: "calib"
- board text added: "dac"
- board text added: "de"
- board text added: "gnd"
- board text added: "scl"
- board text added: "sda"
- board text added: "sig"
- board text added: "uart"
- board text added: "ubd"

Commit message: kicad changes
Parts:
- removed J2: Au+2, 4022S:Au_Electrode
- removed J5: Au-2, 4022S:Au_Electrode
- added C17: 10n, Capacitor_SMD:C_0402_1005Metric, F.Cu at (130.8, 69.0)
- added C18: 10n, Capacitor_SMD:C_0402_1005Metric, F.Cu at (117.2, 75.8)
- added C19: 10n, Capacitor_SMD:C_0402_1005Metric, F.Cu at (116.0, 75.8)
- added C20: 10n, Capacitor_SMD:C_0402_1005Metric, F.Cu at (134.2, 71.8)
- added C21: 10n, Capacitor_SMD:C_0402_1005Metric, F.Cu at (135.4, 71.8)
- added J11: Ti-2, Connector_PinHeader_2.54mm:PinHeader_1x01_P2.54mm_Vertical, B.Cu at (142.5, 93.8)
- added U10: OP07C, Package_SO:SOIC-8_3.9x4.9mm_P1.27mm, F.Cu at (105.0, 94.0)
- added U11: ~, Package_SO:TSSOP-14_4.4x5mm_P0.65mm, F.Cu at (113.0, 94.5)
- J1: value Au+1 -> Au+
- J4: value Au-1 -> Au-
- moved C14 9.13 mm to (125.0, 83.0)
- moved U7 9.13 mm to (125.0, 85.6)
- moved J7 6.49 mm to (138.8, 93.8)
- moved J3 6.14 mm to (146.2, 93.8)
- moved J4 0.65 mm to (130.9, 94.0)
- moved J6 0.40 mm to (135.0, 93.8)
- moved J1 0.29 mm to (118.6, 94.0)
Connections:
- U2 pad 2: unconnected-(U2-PC13-Pad2) -> /SW_Shield+_Au-
- U2 pad 26: /LED_RED -> /Calibration
- U2 pad 27: /LED_GREEN -> /LED_RED
- U2 pad 28: unconnected-(U2-PB2-Pad28) -> /LED_GREEN
- U2 pad 3: unconnected-(U2-PC14-Pad3) -> /SW_Shield-_Au+
- U2 pad 4: unconnected-(U2-PC15-Pad4) -> /SW_Shield-_Au-
- U2 pad 41: /Calibration -> unconnected-(U2-PA8-Pad41)
- U2 pad 53: unconnected-(U2-PC12-Pad53) -> /SW_Shield+_Au+
Routing:
- net /SW_Shield+_Au+: track 0.00 -> 40.0 mm, vias 0 -> 4
- net /SW_Shield+_Au-: track 0.00 -> 38.9 mm, vias 0 -> 2
- net /SW_Shield-_Au+: track 0.00 -> 38.3 mm, vias 0 -> 2
- net /Au- Shield: track 0.00 -> 34.9 mm, vias 0 -> 5
- net /SW_Shield-_Au-: track 0.00 -> 33.4 mm, vias 0 -> 2
- net /Au+ Shield: track 0.00 -> 30.1 mm, vias 0 -> 3
- net /Shield+: track 0.00 -> 19.4 mm
- net GND: track 85.2 -> 101.6 mm, vias 19 -> 25
- net /Calibration: track 71.1 -> 82.0 mm, vias 4 -> 7
- net /SDA: track 98.4 -> 88.0 mm, vias 6 -> 4
- net /AMP: track 100.1 -> 109.8 mm
- net /SCL: track 98.3 -> 89.4 mm, vias 7 -> 5
- net /Ti-: track 68.3 -> 61.5 mm
- net /Au-: track 68.2 -> 62.5 mm, vias 4 -> 3
- net /DAC: track 55.2 -> 60.7 mm
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Other:
- board text added: "Author: Cameron Clark University of Cape Town Salinometer Controller Board v0 22/08/2024"

Commit message: heading for lit review
Parts:
- added C22: 10u, Capacitor_SMD:C_0603_1608Metric, F.Cu at (106.7, 59.5)
- U1: value ~ -> DAC53401
- U11, U3, U6, U8: value ~ -> 4xSwitch
- U7: value ~ -> TempSensor
- U9: value ~ -> DepthSensor
Routing:
- net +3V3: track 64.0 -> 67.8 mm
- net GND: track 101.6 -> 103.4 mm
Other:
- outline, holes or cut-outs redrawn
